File: rectificador.sch (KiCad schematic (older format))
At the start: 134 parts, among them J1 TRIF, J10 AC_FASE_2, J11 AC_FASE_3, J12 SEC, J13 BOB_CONT, J14 PUENTE_P, J15 PUENTE_N, J16 RES_LIM, J17 CONTACT, J18 INDUCT, J19 MCU, J2 CHASIS, J21 VENT, J22 TC, J3 PRIM, J4 FILTRO_1, J5 FILTRO_2, J6 FILTRO_3, J7 BUS, J8 COM, J9 AC_FASE_1, K1 SRD-05VDC-SLC, Q1 2n2222, Q2 MMBT3904, U1 LM7805_TO220, U2 PC817, U3 PC817, U4 ACS712xLCTR-30A, U5 AMC1301, U6 LM358, U7 MAX6675, U8 220VAC_5VD_SWITCHING, U9 PC817

Commit message: actualizo valores de componentes
Parts:
- C19: value 10uF/10V -> 47uF/25V
- C29: value 10uFx10V -> 47uFx25V
- C31: value 47uFx25V -> 47uFx25V/NP
- D10: value 2V4 -> 2V4/NP
- D5: value LED_NA -> LED_AZ; parte (none) -> Kingbright std led 470nm blue APT1608QBC
- JP1: value MCU/AUTO -> MCU/AUTO-NP
- K1: parte (none) -> Songle relay SRD-05VDC-SL-C
- Q2: value MMBT3904 -> MMBT3904/NP
- R12: value 1K -> 1K/NP
- R19: value 1K -> NP
- R2: value 470 -> 470/NP
- R5: value 390 -> 220; parte (none) -> Yageo thick film resistor RC0603JR-07220RL 220ohm 5%
- U4: Parte (none) -> Allegro ACS712T-ELC-30A
Other:
- note added: "foot_err\n"
Changed lines of the file:
@@
 AR Path="/5C36DB72" Ref="D5"  Part="1"
 F 0 "D5" V 3950 3725 50  0000 C CNN
-F 1 "LED_NA" V 4025 3775 50  0000 C CNN
+F 1 "LED_AZ" V 4025 3775 50  0000 C CNN
 F 2 "LED_SMD:LED_0603_1608Metric_Pad1.05x0.95mm_HandSolder" V 3950 3575 50  0001 C CNN
 F 3 "~" V 3950 3575 50  0001 C CNN
+F 4 "Kingbright std led 470nm blue APT1608QBC" V 3950 3575 50  0001 C CNN "parte"
 	1    3950 3575
 	0    1    1    0
@@
 AR Path="/5C502414" Ref="R2"  Part="1"
 F 0 "R2" H 5866 4029 50  0000 R CNN
-F 1 "470" H 5866 4120 50  0000 R CNN
+F 1 "470/NP" H 5866 4120 50  0000 R CNN
 F 2 "Resistor_SMD:R_0603_1608Metric_Pad1.05x0.95mm_HandSolder" H 5925 4075 50  0001 C CNN
 F 3 "~" H 5925 4075 50  0001 C CNN
@@
 F 2 "Package_SO:SOIC-8_3.9x4.9mm_P1.27mm" H 7250 1325 50  0001 L CIN
 F 3 "E:\\biblioteca\\hojas_de_datos\\Sensado de corriente con shunt\\hall_effect\\ACS712-Datasheet.pdf" H 7150 1675 50  0001 C CNN
+F 4 "Allegro ACS712T-ELC-30A" V 7150 1675 50  0001 C CNN "Parte"
 	1    7150 1675
 	0    1    1    0
@@
 AR Path="/5C2B98C5/5D34C209" Ref="C?"  Part="1"
 F 0 "C19" H 7650 5775 50  0000 L CNN
-F 1 "10uF/10V" H 7650 5675 50  0000 L CNN
+F 1 "47uF/25V" H 7650 5675 50  0000 L CNN
 F 2 "arias2015:CP_Radial_D6.3mm_P2.50mm" H 7600 5875 50  0001 C CNN
 F 3 "~" H 7600 5875 50  0001 C CNN
@@
 AR Path="/5C2B98C5/5D34C253" Ref="C?"  Part="1"
 F 0 "C29" H 10241 5671 50  0000 L CNN
-F 1 "10uFx10V" H 10200 5525 50  0000 L CNN
+F 1 "47uFx25V" H 10200 5525 50  0000 L CNN
 F 2 "arias2015:CP_Radial_D6.3mm_P2.50mm" H 10150 5625 50  0001 C CNN
 F 3 "~" H 10150 5625 50  0001 C CNN
@@
 F 2 "arias2015:Relay_SPDT_SANYOU_SRD_Series_Form_C" H 3825 2800 60  0001 C CNN
 F 3 "E:\\biblioteca\\hojas_de_datos\\rele\\Rele_SRD_subminiature_high_power_realy.pdf" H 3825 2800 60  0001 C CNN
+F 4 "Songle relay SRD-05VDC-SL-C" H 3475 2900 50  0001 C CNN "parte"
 	1    3475 2900
 	-1   0    0    -1
@@
 AR Path="/5C2B98C5/5DEFAA45" Ref="R?"  Part="1"
 F 0 "R5" V 6075 3300 50  0000 C CNN
-F 1 "390" V 6150 3300 50  0000 C CNN
+F 1 "220" V 6150 3300 50  0000 C CNN
 F 2 "Resistor_SMD:R_0603_1608Metric_Pad1.05x0.95mm_HandSolder" H 6225 3300 50  0001 C CNN
 F 3 "~" H 6225 3300 50  0001 C CNN
+F 4 "Yageo thick film resistor RC0603JR-07220RL 220ohm 5%" V 6225 3300 50  0001 C CNN "parte"
 	1    6225 3300
 	0    1    1    0
@@
 P 5475 3875
 F 0 "Q2" H 5350 4050 50  0000 C CNN
-F 1 "MMBT3904" H 5200 3975 50  0000 C CNN
+F 1 "MMBT3904/NP" H 5150 3975 50  0000 C CNN
 F 2 "Package_TO_SOT_SMD:SOT-23" H 5675 3800 50  0001 L CIN
 F 3 "https://www.fairchildsemi.com/datasheets/2N/2N3904.pdf" H 5475 3875 50  0001 L CNN
@@
 P 6200 3875
 F 0 "D10" H 6075 3925 50  0000 C CNN
-F 1 "2V4" H 6075 3825 50  0000 C CNN
+F 1 "2V4/NP" H 6150 3800 50  0000 C CNN
 F 2 "arias2015:D_DO-35_SOD27_P7.62mm_Horizontal" V 6200 3875 50  0001 C CNN
 F 3 "~" V 6200 3875 50  0001 C CNN
@@
 AR Path="/5D091234" Ref="C31"  Part="1"
 F 0 "C31" H 6650 4050 50  0000 L CNN
-F 1 "47uFx25V" H 6625 3950 50  0000 L CNN
+F 1 "47uFx25V/NP" H 6625 3950 50  0000 L CNN
 F 2 "arias2015:CP_Radial_D6.3mm_P2.50mm" H 6525 4050 50  0001 C CNN
 F 3 "~" H 6525 4050 50  0001 C CNN
@@
 AR Path="/5C2B98C5/5D1D7C98" Ref="R?"  Part="1"
 F 0 "R12" H 6400 3625 50  0000 C CNN
-F 1 "1K" H 6400 3550 50  0000 C CNN
+F 1 "1K/NP" H 6350 3550 50  0000 C CNN
 F 2 "Resistor_SMD:R_0603_1608Metric_Pad1.05x0.95mm_HandSolder" H 6525 3625 50  0001 C CNN
 F 3 "~" H 6525 3625 50  0001 C CNN
@@
 P 5175 3800
 F 0 "JP1" V 5525 3800 50  0000 L CNN
-F 1 "MCU/AUTO" V 5600 3800 50  0000 L CNN
+F 1 "MCU/AUTO-NP" V 5600 3800 50  0000 L CNN
 F 2 "arias2015:PinHeader_1x03_P2.54mm_Vertical" H 5175 3800 50  0001 C CNN
 F 3 "~" H 5175 3800 50  0001 C CNN
@@
 AR Path="/5CFBB453" Ref="R19"  Part="1"
 F 0 "R19" H 4925 4025 50  0000 R CNN
-F 1 "1K" H 4950 3950 50  0000 R CNN
+F 1 "NP" H 4950 3950 50  0000 R CNN
 F 2 "Resistor_SMD:R_0603_1608Metric_Pad1.05x0.95mm_HandSolder" H 5000 4000 50  0001 C CNN
 F 3 "~" H 5000 4000 50  0001 C CNN
@@
 Text Notes 5225 6300 0    50   ~ 0
 8mA\n
+Text Notes 4225 4025 0    50   Italic 10
+foot_err\n
 $EndSCHEMATC
